Commit message: make robots move

File: src/my_r2d2/urdf/r2d2.urdf.xacro (robot description, xacro)
@@ -23,4 +23,10 @@
     </inertial>
   </xacro:macro>
+  <link name="base_footprint"/>
+  <joint name="base_footprint_joint" type="fixed">
+    <parent link="base_footprint"/>
+    <child link="base_link"/>
+    <origin xyz="0 0 0.47" rpy="0 0 0"/>
+  </joint>
   <link name="base_link">
     <visual>

Commit message: ar camera

File: src/my_r2d2/urdf/r2d2.urdf.xacro (robot description, xacro)
@@ -219,3 +219,17 @@
     <origin xyz="${.707*width+0.04} 0 ${.707*width}"/>
   </joint>
+  <link name="eye">
+    <visual>
+      <geometry>
+        <box size="0.03 0.01 0.03"/>
+      </geometry>
+      <origin xyz="0 0 0" rpy="0 0 0"/>
+      <material name="black"/>
+    </visual>
+  </link>
+  <joint name="toeye" type="fixed">
+    <parent link="box" />
+    <child link="eye" />
+    <origin xyz="0 0 0" rpy="${-pi/2} 0 ${-pi/2}"/>
+  </joint>
 </robot>
